Commit message: nouvelle tentative de configuration manuelle

File: src/franka_sonde/urdf/fr3_sur_rail.xacro (robot description, xacro)
@@ -26,5 +26,4 @@
     <parent link="montage"/>
     <child link="base"/>
-    <origin xyz="0 0 0" rpy="0 0 0"/>
   </joint>
 </robot>

File: src/franka_sonde/urdf/sonde_robot_rail.xacro (robot description, xacro)
@@ -51,5 +51,5 @@
       <command_interface name="position">
         <param name="min">0.0</param>
-        <param name="max">2.0</param>
+        <param name="max">1.7</param>
       </command_interface>
       <state_interface name="position">
