Commit message: A - etape 1

File: src/franka_sonde/urdf/rail_sur_table.xacro (robot description, xacro)
@@ -60,12 +60,10 @@
     </inertial>
   </link>
-  <joint name="rail_joint" type="$(arg rail_joint_type)">
+  <joint name="rail_joint" type="prismatic">
     <origin xyz="0 -0.85 0" rpy="0 0 0"/>
     <parent link="rail"/>
     <child link="montage"/>
-    <xacro:if value="${'$(arg rail_joint_type)' == 'prismatic'}">
-      <axis xyz="0 1 0"/>
-      <limit lower="0" upper="1.7" effort="1000" velocity="0.5"/>
-    </xacro:if>
+    <axis xyz="0 1 0"/>
+    <limit lower="0" upper="1.7" effort="1000" velocity="0.5"/>
   </joint>
 </robot>

File: src/franka_sonde/urdf/srr.xacro (robot description, xacro)
@@ -33,8 +33,4 @@
   <xacro:arg name="ee_id"           default="none"/>
   <xacro:arg name="gazebo_effort"   default="false"/>
-  <!-- fixed : la chaîne KDL n'a que 7 joints mobiles (FR3)
-       → JntToGravity reçoit un vecteur de taille 7 = OK
-       prismatic ajouterait un 8e joint → taille mismatch → ERROR -->
-  <xacro:arg name="rail_joint_type" default="fixed"/>
   <!-- =============================================
        BRAS FR3
@@ -124,4 +120,23 @@
     <origin xyz="0 0 0.2" rpy="0 0 0"/>
   </joint>
+  <!-- =============================================
+       RAIL — ros2_control
+       Plugin standard ign_ros2_control (même base que Franka).
+       Bloc séparé → hardware interface indépendante sous le même CM.
+       La chaîne KDL du bras commence à fr3_link0 → ce joint n'est
+       pas vu par l'IK, il est commandé séparément (rail_controller).
+  ============================================= -->
+  <ros2_control name="RailSystem" type="system">
+    <hardware>
+      <plugin>franka_ign_ros2_control/IgnitionSystem</plugin>
+    </hardware>
+    <joint name="rail_joint">
+      <command_interface name="position"/>
+      <state_interface name="position">
+        <param name="initial_value">0.0</param>
+      </state_interface>
+      <state_interface name="velocity"/>
+    </joint>
+  </ros2_control>
   <!-- RailSystem supprimé :
        mock_components/GenericSystem est incompatible avec

Commit message: nouvelle position du rail au launch

File: src/franka_sonde/urdf/rail_sur_table.xacro (robot description, xacro)
@@ -3,5 +3,7 @@
   <!-- rail_joint_type : "fixed" pour Gazebo (7 DOF → gravity comp OK)
                          "prismatic" pour RViz / visualisation standalone -->
-  <xacro:arg name="rail_joint_type" default="prismatic"/>
+  <!-- Position initiale du rail (m) — passée depuis le launch file.
+       Le joint est fixe pour compatibilité avec FrankaHardwareInterface/KDL. -->
+  <xacro:arg name="rail_position" default="0.0"/>
   <!-- Table (root link - KDL doesn't support inertia here, but Gazebo needs a small mass) -->
   <link name="table">
@@ -60,10 +62,8 @@
     </inertial>
   </link>
-  <joint name="rail_joint" type="prismatic">
-    <origin xyz="0 -0.85 0" rpy="0 0 0"/>
+  <joint name="rail_joint" type="fixed">
+    <origin xyz="0 ${-0.85 + $(arg rail_position)} 0" rpy="0 0 0"/>
     <parent link="rail"/>
     <child link="montage"/>
-    <axis xyz="0 1 0"/>
-    <limit lower="0" upper="1.7" effort="1000" velocity="0.5"/>
   </joint>
 </robot>

File: src/franka_sonde/urdf/srr.xacro (robot description, xacro)
@@ -33,4 +33,5 @@
   <xacro:arg name="ee_id"           default="none"/>
   <xacro:arg name="gazebo_effort"   default="false"/>
+  <xacro:arg name="rail_position"   default="0.0"/>
   <!-- =============================================
        BRAS FR3
@@ -120,30 +121,5 @@
     <origin xyz="0 0 0.2" rpy="0 0 0"/>
   </joint>
-  <!-- =============================================
-       RAIL — ros2_control
-       Plugin standard ign_ros2_control (même base que Franka).
-       Bloc séparé → hardware interface indépendante sous le même CM.
-       La chaîne KDL du bras commence à fr3_link0 → ce joint n'est
-       pas vu par l'IK, il est commandé séparément (rail_controller).
-  ============================================= -->
-  <ros2_control name="RailSystem" type="system">
-    <hardware>
-      <plugin>franka_ign_ros2_control/IgnitionSystem</plugin>
-    </hardware>
-    <joint name="rail_joint">
-      <command_interface name="position"/>
-      <state_interface name="position">
-        <param name="initial_value">0.0</param>
-      </state_interface>
-      <state_interface name="velocity"/>
-    </joint>
-  </ros2_control>
-  <!-- RailSystem supprimé :
-       mock_components/GenericSystem est incompatible avec
-       franka_ign_ros2_control/IgnitionSystem (base class différente).
-       Le rail_joint est laissé sans interface ros2_control pour l'instant.
-       Son état est fourni par joint_state_publisher dans le launch file. -->
-  <!-- fr3_arm_controller est enregistré via spawner avec param-file
-       dans le launch file, pas ici, pour eviter un second
-       controller_manager. -->
+  <!-- rail_joint injecté dans FrankaHardwareInterface via le launch file
+       (même plugin IgnitionSystem, seule solution compatible Gazebo) -->
 </robot>
